File: ai-3-pcb-guide.kicad_pcb (KiCad board)
At the start: 2 copper layers, 21 parts, among them SW1 SW_Push

Commit message: edit
Parts:
- added F1: 500mA, Fuse_Holders_and_Fuses:Fuse_SMD1206_Reflow, F.Cu at (304.8, 38.1)
- added U1: ATmega32U4-AU, Housings_QFP:TQFP-44_10x10mm_Pitch0.8mm, F.Cu at (138.8, 47.6)
- added Y1: 16Mhz, Crystals:Crystal_SMD_3225-4pin_3.2x2.5mm, F.Cu at (133.5, 37.2)
- moved D1 168.9 mm to (172.7, 38.1), turned to 90 degrees
- moved D3 167.6 mm to (172.7, 58.4), turned to 90 degrees
- moved MX3 166.1 mm to (165.1, 58.4)
- moved D2 163.1 mm to (193.0, 38.1), turned to 90 degrees
- moved D4 149.6 mm to (193.0, 58.4), turned to 90 degrees
- moved MX1 140.2 mm to (165.1, 38.1)
- moved MX4 140.2 mm to (185.4, 58.4)
- moved MX2 115.7 mm to (185.4, 38.1)
- moved USB1 59.9 mm to (340.4, 48.3)
- moved C2 28.3 mm to (335.3, 0.00)
- moved R1 23.0 mm to (353.1, 5.08)
- moved R3 20.2 mm to (363.2, 5.08)
- moved C6 19.4 mm to (355.6, 0.00)
- moved R4 15.2 mm to (368.3, 5.08)
- moved R2 14.1 mm to (358.1, 5.08)
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